File: Schematics/HackenTop-BreakoutTest/HackenTop-BreakoutTest.sch (KiCad schematic (older format))
At the start: 27 parts

Commit message: Starting routing
Parts:
- removed J?: Conn_01x06, symbol Connector_Generic:Conn_01x06
- added C1, C3: 47uF, Capacitor_SMD:C_0805_2012Metric, symbol Device:C_Small
- added C6, C9: 100nF, Capacitor_SMD:C_0805_2012Metric, symbol Device:C_Small
- added D1: Activity, LED_SMD:LED_0603_1608Metric, symbol Device:LED_Small
- added J2: Conn_01x07, Connector_PinHeader_2.54mm:PinHeader_1x07_P2.54mm_Vertical, symbol Connector_Generic:Conn_01x07
- added J4: Conn_01x03, Connector_PinHeader_2.54mm:PinHeader_1x03_P2.54mm_Vertical, symbol Connector_Generic:Conn_01x03
- added J5: Conn_01x25, Connector_PinHeader_2.54mm:PinHeader_1x25_P2.54mm_Vertical, symbol Connector_Generic:Conn_01x25
- added J6: Conn_01x21, Connector_PinHeader_2.54mm:PinHeader_1x21_P2.54mm_Vertical, symbol Connector_Generic:Conn_01x21
- added J8: Power, TerminalBlock_RND:TerminalBlock_RND_205-00012_1x02_P5.00mm_Horizontal, symbol Connector_Generic:Conn_01x02
- added Q1, Q2, Q3, Q4: 2N7002, HackenTop:DMG1012T, symbol Transistor_FET:2N7002
- added R1: 0ohm, Resistor_SMD:R_0805_2012Metric, symbol Device:R_Small
- added R2: NF, Resistor_SMD:R_0805_2012Metric, symbol Device:R_Small
- added R3: 100k, Resistor_SMD:R_0805_2012Metric, symbol Device:R_Small
- added R4, R5: 47k, Resistor_SMD:R_0805_2012Metric, symbol Device:R_Small
- added R6: 470, Resistor_SMD:R_0805_2012Metric, symbol Device:R_Small
- added U3: ESD5384, HackenTop:ESD5384, symbol HackenTop:ESD5384
- added U4: AP2331W, Package_TO_SOT_SMD:SOT-23, symbol HackenTop:AP2331W
- C10, C12, C14, C7: renamed from C?; footprint (none) -> Capacitor_SMD:C_0805_2012Metric
- D2, D3, D4, D5: renamed from D?; footprint (none) -> LED_SMD:LED_0603_1608Metric
- F1: renamed from F?; footprint (none) -> Fuse:Fuse_1812_4532Metric
- J3: renamed from J?; footprint (none) -> HackenTop:HDMI-jing
- J7: renamed from J?; footprint CONN_1473005-1_TYCO -> HackenTop:TE_1473149-4
- RN1, RN2: renamed from RN?; footprint (none) -> Resistor_SMD:R_Array_Convex_4x0603
- gave numbers to parts that had none: 10
Connections:
- net +1V8: now also J2.2 (Pin_2), R3.1, R5.2
- net +3V3: now also J2.3 (Pin_3), R2.1, R6.1
- net EMMC_DISABLE_N: now also Q3.3 (D)
- net EMMC_EN_N_1V8: now also Q4.1 (G), R5.1
- net GPIO0: now also J5.25 (Pin_25)
- net GPIO1: now also J5.24 (Pin_24)
- net GPIO10: now also J5.13 (Pin_13)
- net GPIO11: now also J5.11 (Pin_11)
- net GPIO12: now also J5.9 (Pin_9)
- net GPIO13: now also J5.7 (Pin_7)
- net GPIO14: now also J5.5 (Pin_5)
- net GPIO15: now also J5.3 (Pin_3)
- net GPIO16: now also J5.1 (Pin_1)
- net GPIO17: now also J6.20 (Pin_20)
- net GPIO18: now also J6.18 (Pin_18)
- net GPIO19: now also J6.16 (Pin_16)
- net GPIO2: now also J5.23 (Pin_23)
- net GPIO20: now also J6.14 (Pin_14)
- net GPIO21: now also J6.12 (Pin_12)
- net GPIO22: now also J6.10 (Pin_10)
- net GPIO23: now also J6.8 (Pin_8)
- net GPIO24: now also J6.6 (Pin_6)
- net GPIO25: now also J6.4 (Pin_4)
- net GPIO26: now also J6.2 (Pin_2)
- net GPIO27: now also J6.1 (Pin_1)
- net GPIO28: now also RN1.1 (R1.1), J5.16 (Pin_16)
- net GPIO29: now also RN1.2 (R2.1), J5.14 (Pin_14)
- net GPIO3: now also J5.22 (Pin_22)
- net GPIO30: now also J5.12 (Pin_12)
- net GPIO31: now also J5.10 (Pin_10)
- net GPIO32: now also J5.8 (Pin_8)
- net GPIO33: now also J5.6 (Pin_6)
- net GPIO34: now also J5.4 (Pin_4)
- net GPIO35: now also J5.2 (Pin_2)
- net GPIO36: now also J6.21 (Pin_21)
- net GPIO37: now also J6.19 (Pin_19)
- net GPIO38: now also J6.17 (Pin_17)
- net GPIO39: now also J6.15 (Pin_15)
- net GPIO4: now also J5.21 (Pin_21)
- net GPIO40: now also J6.13 (Pin_13)
- net GPIO41: now also J6.11 (Pin_11)
- net GPIO42: now also J6.9 (Pin_9)
- net GPIO43: now also J6.7 (Pin_7)
- net GPIO44: now also RN1.3 (R3.1), J6.5 (Pin_5)
- net GPIO45: now also RN1.4 (R4.1), J6.3 (Pin_3)
- net GPIO5: now also J5.20 (Pin_20)
- net GPIO6: now also J5.19 (Pin_19)
- net GPIO7: now also J5.18 (Pin_18)
- net GPIO8: now also J5.17 (Pin_17)
- net GPIO9: now also J5.15 (Pin_15)
- net HDMI_CEC: now also Q2.2 (S), R2.2
- net HDMI_CLK_N: now also J3.12 (CK-)
- net HDMI_CLK_P: now also J3.10 (CK+)
- net HDMI_D0_N: now also J3.9 (D0-)
- net HDMI_D0_P: now also J3.7 (D0+)
- net HDMI_HPD_N_1V8: now also Q1.3 (D), R3.2
- net HDMI_SCL: now also J3.15 (SCL), U3.A3 (SCL)
- net HDMI_SDA: now also J3.16 (SDA), U3.B3 (SDA)
- net RUN: now also J2.6 (Pin_6)
- net VBUS: now also C1.1, C3.1, C6.1, J2.1 (Pin_1), J8.1 (Pin_1), R1.2, U4.3 (IN); no longer F1.1
- net VDD: now also J2.7 (Pin_7)
- net VDDA: now also J2.4 (Pin_4)
- net VSS: now also J3.11 (CKS), J3.17 (GND), J3.2 (D2S), J3.5 (D1S), J3.8 (D0S), J3.SH, C1.2, C3.2, C6.2, C9.2, J2.5 (Pin_5), J4.3 (Pin_3), J8.2 (Pin_2), Q1.2 (S), Q4.2 (S), R4.2, U3.B2 (GND), U3.C2 (GND), U4.1 (GND)
- net at J3.13 (CEC): now also Q2.3 (D), U3.A2 (CEC)
- net +5V: now reaches J3.18 (+5V)
- net +5V: now also C9.1, Q2.1 (G), U3.A1 (5V), U3.C1 (RPU), U4.2 (OUT)
- net at J3.19 (HPD): now also Q1.1 (G), U3.C3 (HPD)
- new net: J4.2 (Pin_2), Q3.1 (G), R4.1
- new net: D1.1 (K), Q3.2 (S), Q4.3 (D)
- new net: D1.2 (A), R6.2
- new net +5VA: F1.1, J4.1 (Pin_1), R1.1
- no-connect marks 19 -> 21
Other:
- note added: "USB boot enable"
- moved on the sheet: C10, C12, C14, C7, F1, J1, RN1

Commit message: V1 ordered May26
Parts:
- removed J5: Conn_01x25, Connector_PinHeader_2.54mm:PinHeader_1x25_P2.54mm_Vertical, symbol Connector_Generic:Conn_01x25
- added D6, D7, D8, D9: LED_Small, LED_SMD:LED_0603_1608Metric, symbol Device:LED_Small
- added R10, R11, R7, R8, R9: 0ohm, Resistor_SMD:R_0805_2012Metric, symbol Device:R_Small
- added RN3: 470ohm, Resistor_SMD:R_Array_Convex_4x0603, symbol Device:R_Pack04
- U5: footprint Package_TO_SOT_SMD:SOT-223-3_TabPin2 -> Package_TO_SOT_SMD:SOT-23
Connections:
- net GPIO28-45_VDD is gone; now on net GPIO0-27_VDD: J7.41, J7.42
- net +1V8: now also R11.2
- net +3V3: now also R10.1, R9.2
- net +5V: now also C14.2, J2.1 (Pin_1), J7.197, J7.198, J7.199, J7.200, RN2.1 (R1.1)
- net +5VA: now also J1.1 (VBUS); no longer F1.1
- net GPIO0: now also RN3.4 (R4.1)
- net GPIO0-27_VDD: now also R10.2, R11.1
- net GPIO1: now also RN3.3 (R3.1)
- net GPIO2: now also RN3.2 (R2.1)
- net GPIO24: now also J6.5 (Pin_5); no longer J6.6 (Pin_6)
- net GPIO3: now also RN3.1 (R1.1)
- net GPIO44: now also J6.6 (Pin_6); no longer J6.5 (Pin_5)
- net USB_OTGID: no longer J1.4 (ID)
- net VBUS: now also F1.2, R8.2; no longer C11.1, C14.2, J2.1 (Pin_1), J7.197, J7.198, J7.199, J7.200, J8.1 (Pin_1), R1.2, RN2.1 (R1.1), U5.1 (IN)
- net VSS: now also D6.1 (K), D7.1 (K), D8.1 (K), D9.1 (K)
- new net: F1.1, R1.2, R7.2
- new net: C11.1, R8.1, R9.1, U5.1 (IN)
- new net: D9.2 (A), RN3.5 (R4.2)
- new net: D8.2 (A), RN3.6 (R3.2)
- new net: D7.2 (A), RN3.7 (R2.2)
- new net: D6.2 (A), RN3.8 (R1.2)
- new net +BATT: J8.1 (Pin_1), R7.1
- no-connect marks 21 -> 43
Other:
- moved on the sheet: C1, C3, C5, C8, F1, R1, U2
